File: Mainboard/KiCad/Omega-Mainboard.kicad_pcb (KiCad board)
At the start: 2 copper layers, 333.4 x 149.9 mm, 248 parts, among them J1 5V, J10 POWER, J11 KEYBOARD, J12 RAM_EXT, J13 ~RST~/~NMI, J14 CBUS, J2 Composite, J3 Audio, J4 S-VIDEO, J5 RGB, J6 Cassette, J7 JOYSTICK_A, J8 JOYSTICK_B, J9 PRINTER, Q1 PN2907A, Q2 PN2907A, U1 Z84C00, U10 D41464, U11 D41464, U12 ATF16V8B, U13 ATF16V8B, U14 ATF16V8B, U15 74HCT670, U16 74HCT670, U17 74HCT670, U18 74HCT670, U19 74F541, U2 82C55, U20 74F541, U21 74F541, U22 74HCT540, U23 74HCT273, U24 74HCT273, U25 74F245, U26 74F245, U27 74HCT175, U28 74HCT157, U29 74HCT157, U3 V9938/V9958, U30 74HCT153, U31 74HCT153, U32 74AHCT138, U33 74AHCT125, U34 74HCT74, U35 74HCT74, U36 74HCT74, U37 74AHCT32, U38 74AHCT32, U39 74AHCT32, U4 YM2149, U40 74HCT30, U41 74HCT30, U42 74LS07, U43 74HCT04, U44 74AHCT02, U45 74HCT00, U46 ADM691A, U47 CXA1645, U48 MCP6281, U49 LM311, U5 RP5C01, U6 SST39SF040, U7 AS6C4008, U8 D41464, U9 D41464, Y1 21.477270MHz, Y2 32768 Hz, Y3 4.433618MHz

Commit message: FIX: Updated again Omega-Mainboard.kicad_pcb with correct omega-components.pretty library links
Parts:
- BT1: footprint My_Components:Battery_Holder_CR2032_Universal -> omega_components:Battery_Holder_CR2032_Universal
- C1, C10, C11, C12, C13, C14, C15, C16, C17, C18, C19, C2, C20, C21, C22, C23, C24, C25, C26, C27, C28, C29, C3, C30, C31, C32, C33, C34, C35, C36, C37, C38, C39, C4, C40, C41, C42, C43, C44, C45, C46, C47, C48, C49, C5, C50, C51, C52, C53, C54, C55, C56, C57, C58, C6, C7, C79, C8, C80, C81, C82, C83, C84, C85, C86, C87, C9, C91, C92, C93, C94, F1: footprint My_Components:Cap_Cer_508 -> omega_components:Cap_Cer_508
- C59, C60, C61, C62, C63, C64: footprint My_Components:Cap_Elec_Radial_10mm -> omega_components:Cap_Elec_Radial_10mm
- C65, C66, C67: footprint My_Components:Cap_Elec_Radial_6.3mm -> omega_components:Cap_Elec_Radial_6.3mm
- C68, C69, C70: footprint My_Components:Cap_Pol_508_3 -> omega_components:Cap_Pol_508_3
- C71, C72, C73, C74, C75, C76, C77, C78: footprint My_Components:Cap_Elec_Radial_5mm -> omega_components:Cap_Elec_Radial_5mm
- C88, C89, C90: footprint My_Components:C_Trim_Murata -> omega_components:C_Trim_Murata
- D1: footprint My_Components:Diode_762 -> omega_components:Diode_762
- HOLE1, HOLE10, HOLE11, HOLE2, HOLE3, HOLE4, HOLE5, HOLE6, HOLE7, HOLE8, HOLE9: footprint My_Components:Hole_3mm -> omega_components:Hole_3mm
- J1: footprint My_Components:Conn_Power_Jack_Circular_Pads -> omega_components:Conn_Power_Jack_Circular_Pads
- J10: footprint My_Components:Conn_Friction_Lock_8P_2.54mm -> omega_components:Conn_Friction_Lock_8P_2.54mm
- J11: footprint My_Components:Conn_Pin_Header_8x2_2.54mm -> omega_components:Conn_Pin_Header_8x2_2.54mm
- J12: footprint My_Components:Conn_Pin_Header_20x2_2.54mm -> omega_components:Conn_Pin_Header_20x2_2.54mm
- J13: footprint My_Components:Conn_Pin_Header_2x2_2.54mm -> omega_components:Conn_Pin_Header_2x2_2.54mm
- J14: footprint My_Components:Conn_Pin_Header_13x1_2.54mm -> omega_components:Conn_Pin_Header_13x1_2.54mm
- J2: footprint My_Components:Conn_RCA_Right -> omega_components:Conn_RCA_Composite
- J3: footprint My_Components:Conn_RCA_Right -> omega_components:Conn_RCA_Audio
- J4: footprint My_Components:Conn_Mini_DIN_4pin -> omega_components:Conn_Mini_DIN_4pin
- J5, J6: footprint My_Components:Conn_DIN_8pin -> omega_components:Conn_DIN_8pin
- J7, J8: footprint My_Components:Conn_Dsub_DE9M -> omega_components:Conn_Dsub_DE9M
- J9: footprint My_Components:Conn_Micro_Ribbon_14F -> omega_components:Conn_Micro_Ribbon_14F
- JP1, JP2: footprint My_Components:Conn_Pin_Header_2x1_2.54mm -> omega_components:Conn_Pin_Header_2x1_2.54mm
- JP3, JP4, JP5, JP6: footprint My_Components:Conn_Pin_Header_3x1_2.54mm -> omega_components:Conn_Pin_Header_3x1_2.54mm
- JP7, JP8: footprint My_Components:Conn_Pin_Header_2x3_2.54mm -> omega_components:Conn_Pin_Header_2x3_2.54mm
- L1, L2, L3, R1, R10, R11, R12, R13, R14, R15, R16, R17, R18, R19, R2, R20, R21, R22, R23, R24, R25, R26, R27, R28, R29, R3, R30, R31, R32, R33, R34, R35, R36, R37, R38, R39, R4, R40, R41, R42, R43, R44, R45, R46, R47, R48, R5, R6, R7, R8, R9: footprint My_Components:Res_762 -> omega_components:Res_762
- Q1, Q2: footprint My_Components:Transistor_TO92_EBC_254 -> omega_components:Transistor_TO92_EBC_254
- RR1, RR2, RR3, RR4, RR5, RR6, RR7: footprint My_Components:Conn_SIL10 -> omega_components:Conn_SIL10
- RR10, RR8, RR9: footprint My_Components:Conn_SIL6 -> omega_components:Conn_SIL6
- RY1: footprint My_Components:Relay_SPDT -> omega_components:Relay_SPDT
- SLOT1, SLOT2: footprint My_Components:Conn_Edge_50P -> omega_components:Conn_Edge_50P
- U1, U2, U4: footprint My_Components:IC_DIP40_600 -> omega_components:IC_DIP40_600
- U10, U11, U5, U8, U9: footprint My_Components:IC_DIP18_300 -> omega_components:IC_DIP18_300
- U12, U13, U14, U19, U20, U21, U22, U23, U24, U25, U26: footprint My_Components:IC_DIP20_300 -> omega_components:IC_DIP20_300
- U15, U16, U17, U18, U27, U28, U29, U30, U31, U32, U46: footprint My_Components:IC_DIP16_300 -> omega_components:IC_DIP16_300
- U3: footprint My_Components:IC_SDIP64_600 -> omega_components:IC_SDIP64_600
- U33, U34, U35, U36, U37, U38, U39, U40, U41, U42, U43, U44, U45: footprint My_Components:IC_DIP14_300 -> omega_components:IC_DIP14_300
- U47: footprint My_Components:IC_DIP24_400 -> omega_components:IC_DIP24_400
- U48, U49: footprint My_Components:IC_DIP8_300 -> omega_components:IC_DIP8_300
- U6, U7: footprint My_Components:IC_DIP32_600 -> omega_components:IC_DIP32_600
- Y1, Y3: footprint My_Components:Crystal_HC-49U_Vert -> omega_components:Crystal_HC-49U_Vert
- Y2: footprint My_Components:Crystal_32K_Horiz -> omega_components:Crystal_32K_Horiz
Connections:
- J5 pad ~: GND -> (no net)
- J6 pad ~: GND -> (no net)
